Commit message: change camera pos

File: cliport/environments/assets/ur5/workspace.urdf (robot description, URDF)
Before this commit: robot workspace.urdf, 1 links, 0 joints
Links:
- link baseLink: geometry visual mesh filename=plane.obj scale=0.0155 0.028 1

Commit message: change camera pos

File: cliport/environments/assets/ur5/workspace.urdf (robot description, URDF)
Before this commit: robot workspace.urdf, 1 links, 0 joints
Links:
- link baseLink: geometry visual mesh filename=plane.obj scale=0.0167 0.027 1
