Commit message: modify assets

File: cliport/environments/assets/block/block.urdf (robot description, URDF)
Before this commit: robot box.urdf, 1 links, 0 joints
Links:
- link baseLink: geometry collision box size=0.12 0.12 0.12; visual box size=0.12 0.12 0.12

File: cliport/environments/assets/bowl/bowl.urdf (robot description, URDF)
Before this commit: robot bowl.urdf, 1 links, 0 joints
Links:
- link baseLink: geometry collision mesh filename=cup.obj scale=1.875 1.875 0.375; visual mesh filename=textured-0008192.obj scale=1.875 1.875 0.375

File: cliport/environments/assets/ur5/workspace.urdf (robot description, URDF)
Before this commit: robot workspace.urdf, 1 links, 0 joints
Links:
- link baseLink: geometry visual mesh filename=plane.obj scale=0.0167 0.035 1
